Commit message: fix

File: urdf/spina_robot.urdf (robot description, URDF)
Before this commit: robot modular_spine_robot, 7 links, 6 joints
Links:
- removed link module1
- removed link module2
- removed link module3
- removed link module4
- removed link module5
- removed link module6
- added link module1_link, mass 0.8; collision cylinder length=0.15 radius=0.1; visual cylinder length=0.15 radius=0.1
- added link module1_pitch_link
- added link module1_roll_link
- added link module2_link, mass 0.8; collision cylinder length=0.15 radius=0.1; visual cylinder length=0.15 radius=0.1
- added link module2_pitch_link
- added link module2_roll_link
- added link module3_link, mass 0.8; collision cylinder length=0.15 radius=0.1; visual cylinder length=0.15 radius=0.1
- added link module3_pitch_link
- added link module3_roll_link
- added link module4_link, mass 0.8; collision cylinder length=0.15 radius=0.1; visual cylinder length=0.15 radius=0.1
- added link module4_pitch_link
- added link module4_roll_link
- added link module5_link, mass 0.8; collision cylinder length=0.15 radius=0.1; visual cylinder length=0.15 radius=0.1
- added link module5_pitch_link
- added link module5_roll_link
- added link module6_link, mass 0.8; collision cylinder length=0.15 radius=0.1; visual cylinder length=0.15 radius=0.1
- added link module6_pitch_link
- added link module6_roll_link
Joints:
- removed joint joint1
- removed joint joint2
- removed joint joint3
- removed joint joint4
- removed joint joint5
- removed joint joint6
- added joint pitch1: type revolute, parent base_link, child module1_pitch_link, origin xyz=0 0 0.15 rpy=0 0 0, axis 0 1 0, limit lower=-0.5236 upper=0.5236 effort=10 velocity=1.0
- added joint pitch2: type revolute, parent module1_link, child module2_pitch_link, origin xyz=0 0 0.15 rpy=0 0 0, axis 0 1 0, limit lower=-0.5236 upper=0.5236 effort=10 velocity=1.0
- added joint pitch3: type revolute, parent module2_link, child module3_pitch_link, origin xyz=0 0 0.15 rpy=0 0 0, axis 0 1 0, limit lower=-0.5236 upper=0.5236 effort=10 velocity=1.0
- added joint pitch4: type revolute, parent module3_link, child module4_pitch_link, origin xyz=0 0 0.15 rpy=0 0 0, axis 0 1 0, limit lower=-0.5236 upper=0.5236 effort=10 velocity=1.0
- added joint pitch5: type revolute, parent module4_link, child module5_pitch_link, origin xyz=0 0 0.15 rpy=0 0 0, axis 0 1 0, limit lower=-0.5236 upper=0.5236 effort=10 velocity=1.0
- added joint pitch6: type revolute, parent module5_link, child module6_pitch_link, origin xyz=0 0 0.15 rpy=0 0 0, axis 0 1 0, limit lower=-0.5236 upper=0.5236 effort=10 velocity=1.0
- added joint roll1: type revolute, parent module1_pitch_link, child module1_roll_link, origin xyz=0 0 0 rpy=0 0 0, axis 1 0 0, limit lower=-0.5236 upper=0.5236 effort=10 velocity=1.0
- added joint roll2: type revolute, parent module2_pitch_link, child module2_roll_link, origin xyz=0 0 0 rpy=0 0 0, axis 1 0 0, limit lower=-0.5236 upper=0.5236 effort=10 velocity=1.0
- added joint roll3: type revolute, parent module3_pitch_link, child module3_roll_link, origin xyz=0 0 0 rpy=0 0 0, axis 1 0 0, limit lower=-0.5236 upper=0.5236 effort=10 velocity=1.0
- added joint roll4: type revolute, parent module4_pitch_link, child module4_roll_link, origin xyz=0 0 0 rpy=0 0 0, axis 1 0 0, limit lower=-0.5236 upper=0.5236 effort=10 velocity=1.0
- added joint roll5: type revolute, parent module5_pitch_link, child module5_roll_link, origin xyz=0 0 0 rpy=0 0 0, axis 1 0 0, limit lower=-0.5236 upper=0.5236 effort=10 velocity=1.0
- added joint roll6: type revolute, parent module6_pitch_link, child module6_roll_link, origin xyz=0 0 0 rpy=0 0 0, axis 1 0 0, limit lower=-0.5236 upper=0.5236 effort=10 velocity=1.0

Commit message: launch: Add fixed joints for each module in spina_robot.urdf

File: urdf/spina_robot.urdf (robot description, URDF)
Before this commit: robot spine_robot, 19 links, 12 joints
Joints:
- added joint fixed1: type fixed, parent module1_roll_link, child module1_link, origin xyz=0 0 0 rpy=0 0 0
- added joint fixed2: type fixed, parent module2_roll_link, child module2_link, origin xyz=0 0 0 rpy=0 0 0
- added joint fixed3: type fixed, parent module3_roll_link, child module3_link, origin xyz=0 0 0 rpy=0 0 0
- added joint fixed4: type fixed, parent module4_roll_link, child module4_link, origin xyz=0 0 0 rpy=0 0 0
- added joint fixed5: type fixed, parent module5_roll_link, child module5_link, origin xyz=0 0 0 rpy=0 0 0
- added joint fixed6: type fixed, parent module6_roll_link, child module6_link, origin xyz=0 0 0 rpy=0 0 0

Commit message: fix: URDF

File: urdf/spina_robot.urdf (robot description, URDF)
Before this commit: robot spina, 19 links, 18 joints
Links:
- removed link module1_link
- removed link module1_pitch_link
- removed link module1_roll_link
- removed link module2_link
- removed link module2_pitch_link
- removed link module2_roll_link
- removed link module3_link
- removed link module3_pitch_link
- removed link module3_roll_link
- removed link module4_link
- removed link module4_pitch_link
- removed link module4_roll_link
- removed link module5_link
- removed link module5_pitch_link
- removed link module5_roll_link
- removed link module6_link
- removed link module6_pitch_link
- removed link module6_roll_link
- added link module1; visual cylinder length=0.1 radius=0.05
- added link module1_intermediate, mass 0.01
- added link module2; visual cylinder length=0.1 radius=0.05
- added link module2_intermediate, mass 0.01
- added link module3; visual cylinder length=0.1 radius=0.05
- added link module3_intermediate, mass 0.01
- added link module4; visual cylinder length=0.1 radius=0.05
- added link module4_intermediate, mass 0.01
- added link module5; visual cylinder length=0.1 radius=0.05
- added link module5_intermediate, mass 0.01
- added link module6; visual cylinder length=0.1 radius=0.05
- added link module6_intermediate, mass 0.01
- link base_link: geometry 
Joints:
- removed joint fixed1
- removed joint fixed2
- removed joint fixed3
- removed joint fixed4
- removed joint fixed5
- removed joint fixed6
- removed joint pitch1
- removed joint pitch2
- removed joint pitch3
- removed joint pitch4
- removed joint pitch5
- removed joint pitch6
- removed joint roll1
- removed joint roll2
- removed joint roll3
- removed joint roll4
- removed joint roll5
- removed joint roll6
- added joint joint1_x: type revolute, parent base_link, child module1_intermediate, origin xyz=0 0 0.1 rpy=0 0 0, axis 1 0 0, limit lower=-1.57 upper=1.57 effort=10 velocity=1.0
- added joint joint1_y: type revolute, parent module1_intermediate, child module1, origin xyz=0 0 0 rpy=0 0 0, axis 0 1 0, limit lower=-1.57 upper=1.57 effort=10 velocity=1.0
- added joint joint2_x: type revolute, parent module1, child module2_intermediate, origin xyz=0 0 0.1 rpy=0 0 0, axis 1 0 0, limit lower=-1.57 upper=1.57 effort=10 velocity=1.0
- added joint joint2_y: type revolute, parent module2_intermediate, child module2, origin xyz=0 0 0 rpy=0 0 0, axis 0 1 0, limit lower=-1.57 upper=1.57 effort=10 velocity=1.0
- added joint joint3_x: type revolute, parent module2, child module3_intermediate, origin xyz=0 0 0.1 rpy=0 0 0, axis 1 0 0, limit lower=-1.57 upper=1.57 effort=10 velocity=1.0
- added joint joint3_y: type revolute, parent module3_intermediate, child module3, origin xyz=0 0 0 rpy=0 0 0, axis 0 1 0, limit lower=-1.57 upper=1.57 effort=10 velocity=1.0
- added joint joint4_x: type revolute, parent module3, child module4_intermediate, origin xyz=0 0 0.1 rpy=0 0 0, axis 1 0 0, limit lower=-1.57 upper=1.57 effort=10 velocity=1.0
- added joint joint4_y: type revolute, parent module4_intermediate, child module4, origin xyz=0 0 0 rpy=0 0 0, axis 0 1 0, limit lower=-1.57 upper=1.57 effort=10 velocity=1.0
- added joint joint5_x: type revolute, parent module4, child module5_intermediate, origin xyz=0 0 0.1 rpy=0 0 0, axis 1 0 0, limit lower=-1.57 upper=1.57 effort=10 velocity=1.0
- added joint joint5_y: type revolute, parent module5_intermediate, child module5, origin xyz=0 0 0 rpy=0 0 0, axis 0 1 0, limit lower=-1.57 upper=1.57 effort=10 velocity=1.0
- added joint joint6_x: type revolute, parent module5, child module6_intermediate, origin xyz=0 0 0.1 rpy=0 0 0, axis 1 0 0, limit lower=-1.57 upper=1.57 effort=10 velocity=1.0
- added joint joint6_y: type revolute, parent module6_intermediate, child module6, origin xyz=0 0 0 rpy=0 0 0, axis 0 1 0, limit lower=-1.57 upper=1.57 effort=10 velocity=1.0

Commit message: fix: module 1

File: urdf/spina_robot.urdf (robot description, URDF)
Before this commit: robot spine_robot, 13 links, 12 joints
Links:
- removed link module1
- removed link module1_intermediate
- removed link module2
- removed link module2_intermediate
- removed link module3
- removed link module3_intermediate
- removed link module4
- removed link module4_intermediate
- removed link module5
- removed link module5_intermediate
- removed link module6
- removed link module6_intermediate
- added link gimbal_base, mass 0.05
- added link gimbal_roll_link, mass 0.05
- added link top_disk_link, mass 0.1; collision cylinder length=0.02 radius=0.1; visual cylinder length=0.02 radius=0.1
- link base_link: mass 1.0 -> 0.1; geometry collision cylinder length=0.02 radius=0.1; visual cylinder length=0.02 radius=0.1
Joints:
- removed joint joint1_x
- removed joint joint1_y
- removed joint joint2_x
- removed joint joint2_y
- removed joint joint3_x
- removed joint joint3_y
- removed joint joint4_x
- removed joint joint4_y
- removed joint joint5_x
- removed joint joint5_y
- removed joint joint6_x
- removed joint joint6_y
- added joint base_to_gimbal: type fixed, parent base_link, child gimbal_base, origin xyz=0 0 0.075 rpy=0 0 0
- added joint gimbal_pitch: type revolute, parent gimbal_base, child gimbal_roll_link, origin xyz=0 0 0 rpy=0 0 0, axis 0 1 0, limit lower=-3.14 upper=3.14 effort=1 velocity=1
- added joint gimbal_roll: type revolute, parent gimbal_roll_link, child top_disk_link, origin xyz=0 0 0 rpy=0 0 0, axis 1 0 0, limit lower=-3.14 upper=3.14 effort=1 velocity=1

Commit message: fix

File: urdf/spina_robot.urdf (robot description, URDF)
Before this commit: robot two_disk_robot, 4 links, 3 joints
Joints:
- joint gimbal_pitch: limit lower=-3.14 upper=3.14 effort=1 velocity=1 -> lower=-0.5236 upper=0.5236 effort=1 velocity=1
- joint gimbal_roll: limit lower=-3.14 upper=3.14 effort=1 velocity=1 -> lower=-0.5236 upper=0.5236 effort=1 velocity=1

Commit message: fix

File: urdf/spina_robot.urdf (robot description, URDF)
Before this commit: robot spina, 4 links, 3 joints
Links:
- removed link top_disk_link
- added link module1, mass 0.1; collision cylinder length=0.02 radius=0.1; visual cylinder length=0.02 radius=0.1
- added link module2_upper_link, mass 0.1; collision cylinder length=0.02 radius=0.1; visual cylinder length=0.02 radius=0.1
- link base_link: mass 0.1 -> None; geometry 
Joints:
- added joint base_to_module1: type fixed, parent base_link, child module1, origin xyz=0 0 0 rpy=0 0 0
- joint base_to_gimbal: parent base_link -> module1
- joint gimbal_roll: child top_disk_link -> module2_upper_link

Commit message: fix

File: urdf/spina_robot.urdf (robot description, URDF)
Before this commit: robot spina, 5 links, 4 joints
Links:
- removed link gimbal_base
- removed link gimbal_roll_link
- removed link module1
- added link gimbal_pich_link, mass 0.05
- added link module1_gimbal_base, mass 0.05
- added link module1_lower_link, mass 0.1; collision cylinder length=0.02 radius=0.1; visual cylinder length=0.02 radius=0.1
Joints:
- removed joint base_to_module1
- added joint base_link_TO_module1_lower_link: type fixed, parent base_link, child module1_lower_link, origin xyz=0 0 0 rpy=0 0 0
- joint base_to_gimbal: child gimbal_base -> module1_gimbal_base; parent module1 -> module1_lower_link
- joint gimbal_pitch: child gimbal_roll_link -> gimbal_pich_link; parent gimbal_base -> module1_gimbal_base
- joint gimbal_roll: parent gimbal_roll_link -> gimbal_pich_link

Commit message: fix

File: urdf/spina_robot.urdf (robot description, URDF)
Before this commit: robot spina, 5 links, 4 joints
Links:
- removed link gimbal_pich_link
- removed link module1_gimbal_base
- added link module1_pich_link, mass 0.05
- added link module1_roll_link, mass 0.05
Joints:
- removed joint base_to_gimbal
- removed joint gimbal_pitch
- added joint module1_gimbal_pitch: type revolute, parent module1_roll_link, child module1_pich_link, origin xyz=0 0 0 rpy=0 0 0, axis 0 1 0, limit lower=-0.5236 upper=0.5236 effort=1 velocity=1
- added joint module1_gimbal_roll: type revolute, parent module1_lower_link, child module1_roll_link, origin xyz=0 0 0.075 rpy=0 0 0, axis 1 0 0, limit lower=-0.5236 upper=0.5236 effort=1 velocity=1
- joint gimbal_roll: parent gimbal_pich_link -> module1_pich_link

Commit message: fix: finish module1

File: urdf/spina_robot.urdf (robot description, URDF)
Before this commit: robot spina, 5 links, 4 joints
Links:
- removed link module2_upper_link
- added link module1_upper_link, mass 0.1; collision cylinder length=0.02 radius=0.1; visual cylinder length=0.02 radius=0.1
Joints:
- joint gimbal_roll: axis 1 0 0 -> (none); child module2_upper_link -> module1_upper_link; limit lower=-0.5236 upper=0.5236 effort=1 velocity=1 -> (none); origin xyz=0 0 0 rpy=0 0 0 -> xyz=0 0 0.075 rpy=0 0 0; type revolute -> fixed

Commit message: add: module2

File: urdf/spina_robot.urdf (robot description, URDF)
Before this commit: robot spina, 5 links, 4 joints
Links:
- added link module2_lower_link, mass 0.1; collision cylinder length=0.02 radius=0.1; visual cylinder length=0.02 radius=0.1
- added link module2_pich_link, mass 0.05
- added link module2_roll_link, mass 0.05
- added link module2_upper_link, mass 0.1; collision cylinder length=0.02 radius=0.1; visual cylinder length=0.02 radius=0.1
Joints:
- removed joint gimbal_roll
- added joint base_link_TO_module2_lower_link: type fixed, parent module1_upper_link, child module2_lower_link, origin xyz=0 0 0 rpy=0 0 0
- added joint module1_pich_link_TO_module1_upper_link: type fixed, parent module1_pich_link, child module1_upper_link, origin xyz=0 0 0.075 rpy=0 0 0
- added joint module2_gimbal_pitch: type revolute, parent module2_roll_link, child module2_pich_link, origin xyz=0 0 0 rpy=0 0 0, axis 0 1 0, limit lower=-0.5236 upper=0.5236 effort=1 velocity=1
- added joint module2_gimbal_roll: type revolute, parent module2_lower_link, child module2_roll_link, origin xyz=0 0 0.075 rpy=0 0 0, axis 1 0 0, limit lower=-0.5236 upper=0.5236 effort=1 velocity=1
- added joint odule2_pich_link_TO_module2_upper_link: type fixed, parent module2_pich_link, child module2_upper_link, origin xyz=0 0 0.075 rpy=0 0 0

Commit message: add: module3

File: urdf/spina_robot.urdf (robot description, URDF)
Before this commit: robot spina, 9 links, 8 joints
Links:
- added link module3_lower_link, mass 0.1; collision cylinder length=0.02 radius=0.1; visual cylinder length=0.02 radius=0.1
- added link module3_pich_link, mass 0.05
- added link module3_roll_link, mass 0.05
- added link module3_upper_link, mass 0.1; collision cylinder length=0.02 radius=0.1; visual cylinder length=0.02 radius=0.1
Joints:
- added joint base_link_TO_module3_lower_link: type fixed, parent module2_upper_link, child module3_lower_link, origin xyz=0 0 0 rpy=0 0 0
- added joint module3_gimbal_pitch: type revolute, parent module3_roll_link, child module3_pich_link, origin xyz=0 0 0 rpy=0 0 0, axis 0 1 0, limit lower=-0.5236 upper=0.5236 effort=1 velocity=1
- added joint module3_gimbal_roll: type revolute, parent module3_lower_link, child module3_roll_link, origin xyz=0 0 0.075 rpy=0 0 0, axis 1 0 0, limit lower=-0.5236 upper=0.5236 effort=1 velocity=1
- added joint odule3_pich_link_TO_module2_upper_link: type fixed, parent module3_pich_link, child module3_upper_link, origin xyz=0 0 0.075 rpy=0 0 0

Commit message: add: module4

File: urdf/spina_robot.urdf (robot description, URDF)
Before this commit: robot spina, 13 links, 12 joints
Links:
- added link module4_lower_link, mass 0.1; collision cylinder length=0.02 radius=0.1; visual cylinder length=0.02 radius=0.1
- added link module4_pich_link, mass 0.05
- added link module4_roll_link, mass 0.05
- added link module4_upper_link, mass 0.1; collision cylinder length=0.02 radius=0.1; visual cylinder length=0.02 radius=0.1
Joints:
- removed joint odule2_pich_link_TO_module2_upper_link
- removed joint odule3_pich_link_TO_module2_upper_link
- added joint base_link_TO_module4_lower_link: type fixed, parent module3_upper_link, child module4_lower_link, origin xyz=0 0 0 rpy=0 0 0
- added joint module2_pich_link_TO_module2_upper_link: type fixed, parent module2_pich_link, child module2_upper_link, origin xyz=0 0 0.075 rpy=0 0 0
- added joint module3_pich_link_TO_module3_upper_link: type fixed, parent module3_pich_link, child module3_upper_link, origin xyz=0 0 0.075 rpy=0 0 0
- added joint module4_gimbal_pitch: type revolute, parent module4_roll_link, child module4_pich_link, origin xyz=0 0 0 rpy=0 0 0, axis 0 1 0, limit lower=-0.5236 upper=0.5236 effort=1 velocity=1
- added joint module4_gimbal_roll: type revolute, parent module4_lower_link, child module4_roll_link, origin xyz=0 0 0.075 rpy=0 0 0, axis 1 0 0, limit lower=-0.5236 upper=0.5236 effort=1 velocity=1
- added joint module4_pich_link_TO_module4_upper_link: type fixed, parent module4_pich_link, child module4_upper_link, origin xyz=0 0 0.075 rpy=0 0 0

Commit message: add: module5

File: urdf/spina_robot.urdf (robot description, URDF)
Before this commit: robot spina, 17 links, 16 joints
Links:
- added link module5_lower_link, mass 0.1; collision cylinder length=0.02 radius=0.1; visual cylinder length=0.02 radius=0.1
- added link module5_pich_link, mass 0.05
- added link module5_roll_link, mass 0.05
- added link module5_upper_link, mass 0.1; collision cylinder length=0.02 radius=0.1; visual cylinder length=0.02 radius=0.1
Joints:
- added joint base_link_TO_module5_lower_link: type fixed, parent module4_upper_link, child module5_lower_link, origin xyz=0 0 0 rpy=0 0 0
- added joint module5_gimbal_pitch: type revolute, parent module5_roll_link, child module5_pich_link, origin xyz=0 0 0 rpy=0 0 0, axis 0 1 0, limit lower=-0.5236 upper=0.5236 effort=1 velocity=1
- added joint module5_gimbal_roll: type revolute, parent module5_lower_link, child module5_roll_link, origin xyz=0 0 0.075 rpy=0 0 0, axis 1 0 0, limit lower=-0.5236 upper=0.5236 effort=1 velocity=1
- added joint module5_pich_link_TO_module5_upper_link: type fixed, parent module5_pich_link, child module5_upper_link, origin xyz=0 0 0.075 rpy=0 0 0

Commit message: add: module6

File: urdf/spina_robot.urdf (robot description, URDF)
Before this commit: robot spina, 21 links, 20 joints
Links:
- added link module6_lower_link, mass 0.1; collision cylinder length=0.02 radius=0.1; visual cylinder length=0.02 radius=0.1
- added link module6_pich_link, mass 0.05
- added link module6_roll_link, mass 0.05
- added link module6_upper_link, mass 0.1; collision cylinder length=0.02 radius=0.1; visual cylinder length=0.02 radius=0.1
Joints:
- added joint base_link_TO_module6_lower_link: type fixed, parent module5_upper_link, child module6_lower_link, origin xyz=0 0 0 rpy=0 0 0
- added joint module6_gimbal_pitch: type revolute, parent module6_roll_link, child module6_pich_link, origin xyz=0 0 0 rpy=0 0 0, axis 0 1 0, limit lower=-0.5236 upper=0.5236 effort=1 velocity=1
- added joint module6_gimbal_roll: type revolute, parent module6_lower_link, child module6_roll_link, origin xyz=0 0 0.075 rpy=0 0 0, axis 1 0 0, limit lower=-0.5236 upper=0.5236 effort=1 velocity=1
- added joint module6_pich_link_TO_module6_upper_link: type fixed, parent module6_pich_link, child module6_upper_link, origin xyz=0 0 0.075 rpy=0 0 0
